File: Hardware/Main/V1/Main v1.brd (EAGLE design)
At the start: 200.4 x 58.7 mm, 138 parts, among them J1 3A/250V, J2 3A/250V, J3 3A/250V, J4 3A/250V, Q1 2SK3019TL, U1 TAS5825PRHBR, U2 TAS5825PRHBR, U4 LT3042EDDTRPBFDFN-10_DD_LIT

Commit message: main
Parts:
- added C36, C37, C38, C39, C40, C41, C42, C80: 22uF, Capacitor:CAPC2012X110
- moved TP10 0.90 mm to (63.1, 45.7)
- moved C35 0.50 mm to (44.4, 16.9)
- moved R8 0.40 mm to (140.6, 27.4)
- moved R26 0.30 mm to (73.1, 42.2)
- moved TP11 0.10 mm to (43.1, 24.8)
Connections:
- net GND: now also C36.2, C37.2, C38.2, C39.2, C40.2, C41.2, C42.2, C80.2, JP3.1, JP3.2, JP3.3, JP3.4, MP1.1, MP2.1; no longer JP4.1, JP4.2, JP4.3, JP4.4
- net VCC: now also C36.1, C37.1, C38.1, C39.1, C40.1, C41.1, C42.1, C80.1, JP4.1, JP4.2, JP4.3, JP4.4; no longer JP3.1, JP3.2, JP3.3, JP3.4
Routing:
- net DVDD: track 313.8 -> 270.6 mm
- net GND: track 1.43 -> 16.5 mm, vias 437 -> 586
- net VCC: track 172.6 -> 163.3 mm, vias 92 -> 113
- net PDN: track 158.9 -> 154.3 mm
- net SDOUT: track 134.7 -> 133.9 mm
- net SDA: track 168.9 -> 168.0 mm
- net LRCLK: track 162.1 -> 161.4 mm
- net SCL: track 164.3 -> 163.6 mm
- net N$23: track 0.63 -> 0.00 mm
- net N$21: track 0.57 -> 0.00 mm
Other:
- board text added: "/"
- board text added: "2 × 30 W, 2.0 Mode"
- board text added: "2 × TAS5825M"
- board text added: "3V3"
- board text added: "LDO"
- board text added: "⬆️"
- board text added: "⬇️"
