File: Hardware/Main/V1/Main_v1.sch (EAGLE design)
At the start: 138 parts, among them J1 3A/250V, J2 3A/250V, J3 3A/250V, J4 3A/250V, Q1 2SK3019TL, U1 TAS5825PRHBR, U2 TAS5825PRHBR, U4 LT3042EDDTRPBFDFN-10_DD_LIT

Commit message: main
Parts:
- added C36, C37, C38, C39, C40, C41, C42, C80: 22uF, Capacitor:C_CHIP-0805(2012-METRIC)
Connections:
- net GND: now also C36.2, C37.2, C38.2, C39.2, C40.2, C41.2, C42.2, C80.2, JP3.1, JP3.2, JP3.3, JP3.4, MP1.P$1, MP2.P$1; no longer JP4.1, JP4.2, JP4.3, JP4.4
- net VCC: now also C36.1, C37.1, C38.1, C39.1, C40.1, C41.1, C42.1, C80.1, JP4.1, JP4.2, JP4.3, JP4.4; no longer JP3.1, JP3.2, JP3.3, JP3.4
Other:
- moved on the sheet: C45, C46, C47, C48, C49, C50, C51, C52
