File: Hardware/USB-C/V1/USB-C_PURE_v1.sch (EAGLE design)
At the start: 91 parts, among them J1 USB-C31-A-D-VT-CS1, J4 SAMTEC-SLW-104-01-X-SJ, J5 SAMTEC-SLW-104-01-X-SJ, J7 SAMTEC-SLW-104-01-X-SJ, J8 SAMTEC-SLW-104-01-X-SJ, Q1 2N7002-7-F, Q2 AM4825PE, U1 MP2639AGR-Z, U2 ATMEGA328P, U3 TPS2514AQDBVTQ1DBV6_TEX, U4 XC6209F332MR-GSOT-25_TOR, U5 ESD122DMXRDMX3_TEX, U6 ESD122DMXRDMX3_TEX, U7 MAX77962EWJ06+21-100355_MXM, Y1 CSTNE16M0V530000R0

Commit message: V1
Parts:
- removed C52: 270uF, 16SVPG270M:16SVPG270M
- removed CIB: 33pF, Capacitor:C_CHIP-0402(1005-METRIC)
- removed CTMR: 1uF, Capacitor:C_CHIP-0805(2012-METRIC)
- removed LED1: AA2810, AA2810ASURSK:AA2810
- removed LED2, LED3, LED4: EAPL3809WA1, EAPL3809WA1:EAPL3809WA1
- removed Q2: AM4825PE, AM4825PE:AM4825PE
- removed RIB: 40.2K, Resistor:R_CHIP-0402(1005-METRIC)
- removed RILIM: 432K, Resistor:R_CHIP-0402(1005-METRIC)
- removed RISET: 86.6K, Resistor:R_CHIP-0402(1005-METRIC)
- removed RNTC1: 10K NTC, Sensor:NCP18_CHIP-0603(1608-METRIC)
- removed RNTC2: 15K NTC, Sensor:NCP18_CHIP-0603(1608-METRIC)
- removed ROLIM: 44.2K, Resistor:R_CHIP-0402(1005-METRIC)
- removed TPR54: PINHD-1X7, Connector:PINHD-1X7
- added C10: 4.7uF, Capacitor:C_CHIP-0603(1608-METRIC)
- added C13, C16, C38, C39, C40, C41, C42, C47: 22uF, Capacitor:C_CHIP-0805(2012-METRIC)
- added C20, C22: 0.22uF, Capacitor:C_CHIP-0603(1608-METRIC)
- added C25, C26, C27, C36, C37, C49: 1uF, Capacitor:C_CHIP-0805(2012-METRIC)
- added C28: 2.2uF, Capacitor:C_CHIP-0805(2012-METRIC)
- added C29, C30, C31, C32, C33, C35, C46, C48: 100nF, Capacitor:C_CHIP-0402(1005-METRIC)
- added C34: 1uF, Capacitor:C_CHIP-0402(1005-METRIC)
- added C43: 16SVPG270M, 16SVPG270M:16SVPG270M
- added C44: 12nF, Capacitor:C_CHIP-0402(1005-METRIC)
- added C45: 120pF, Capacitor:C_CHIP-0402(1005-METRIC)
- added CN1: (no value), adafruit:JST_2PIN-THM
- added D5, D6, D7, D8: LED_RED, LED:CHIP-ROUND-R_0805
- added IC1: RP2040_QFN56, adafruit_micro:RP2040_QFN56
- added JP1: PINHD-1X2, Connector:PINHD-1X2
- added R12, R13: 5.1K, Resistor:R_CHIP-0402(1005-METRIC)
- added R14, R32: 10k, Resistor:R_CHIP-0402(1005-METRIC)
- added R15: 0.001, Resistor:R_CHIP-2512(6332-METRIC)
- added R24, R26: 5, Resistor:R_CHIP-0402(1005-METRIC)
- added R25: 100, Resistor:R_CHIP-0603(1608-METRIC)
- added R28, R29: 100K, Resistor:R_CHIP-0603(1608-METRIC)
- added R30, R31: 1k, Resistor:R_CHIP-0402(1005-METRIC)
- added RESET1: KMR2, microbuilder:SWITCH_TACT_SMT4.6X2.8
- added TP10, TP4, TP5, TP6, TP7, TP8, TP9: TEST-POINT3X5, SparkFun-Connectors:TEST-POINT3X5
- added TP11, TP12, TP13, TP14, TP2, TP3: TEST-POINT3, SparkFun-Connectors:TEST-POINT3
- added U$1: OSHW-LOGOMINI, SparkFun-Aesthetics:OSHW-LOGOMINI
- added U10, U11: CSD16412Q5ADQJ8, CSD16412Q5A:CSD16412Q5ADQJ8
- added U12: AC103E2FAC_USS, 103AT‐2:AC103E2FAC_USS
- added U13: DRV2605LDGSRDGS0010A, DRV2605LDGSR‎:DRV2605LDGSRDGS0010A
- added U14: XAL4030-472MECXAL4030-472MEC_COC, XAL4030-332MEC:XAL4030-472MECXAL4030-472MEC_COC
- added U15: TPS54335-1ADRCTDRC10_1P65X2P40_TEX, TPS54335:TPS54335-1ADRCTDRC10_1P65X2P40_TEX
- added U17: ATMEGA328P_TQFP, SparkFun-IC-Microcontroller:ATMEGA328P_TQFP
- added U8: IS31FL3195QFN-16_UF_LIT-L, IS31FL3195:IS31FL3195QFN-16_UF_LIT-L
- added U9: BQ28Z610DRZR, BQ28Z610DRZR:BQ28Z610DRZR
- C1, C17, C21, C4: value 1uF -> 22uF
- C11: value 33pF -> 22uF; device Capacitor:C_CHIP-0402(1005-METRIC) -> Capacitor:C_CHIP-0805(2012-METRIC)
- C12: value CNTC -> 22uF; device Capacitor:C_CHIP-0402(1005-METRIC) -> Capacitor:C_CHIP-0805(2012-METRIC)
- C3: value 22uF -> 0.1uF; device Capacitor:C_CHIP-0805(2012-METRIC) -> Capacitor:C_CHIP-0603(1608-METRIC)
- C7: value 22uF -> 0.015uF; device Capacitor:C_CHIP-0805(2012-METRIC) -> Capacitor:C_CHIP-0603(1608-METRIC)
- C8: value 100nF -> 0.015uF; device Capacitor:C_CHIP-0402(1005-METRIC) -> Capacitor:C_CHIP-0603(1608-METRIC)
- C9: value 1uF -> 4.7uF; device Capacitor:C_CHIP-0805(2012-METRIC) -> Capacitor:C_CHIP-0603(1608-METRIC)
- D4: value B330A-13SMA_DIO -> PMEG4050ETP,115; device B330A-13:B330A-13SMA_DIO -> Diode:DIODE_DO-221-AD
- L1: value DR1050-2R2-RDR1050 -> 15uH; device DR1050-2R2-R:DR1050-2R2-RDR1050 -> IHLP4040DZER150M11:IHLP4040DZER150M11IND_IHLP_4040_DZ_VIS
- Q1: value 2N7002-7-F -> 2N7002K-T1
- R10: value 10K -> 12k
- R11: value 10K -> 10k
- R16, R17: value (none) -> 100; device Resistor:R_CHIP-0402(1005-METRIC) -> Resistor:R_CHIP-0603(1608-METRIC)
- R18, R19: value (none) -> 10M
- R3: value 100 -> 0.01; device Resistor:R_CHIP-0402(1005-METRIC) -> Resistor:R_CHIP-2512(6332-METRIC)
- R4: value 2K -> 10; device Resistor:R_CHIP-0402(1005-METRIC) -> Resistor:R_CHIP-0603(1608-METRIC)
- R5: value 93.1K -> 10; device Resistor:R_CHIP-0402(1005-METRIC) -> Resistor:R_CHIP-0603(1608-METRIC)
- R6: value 200 -> 200K; device Resistor:R_CHIP-0402(1005-METRIC) -> Resistor:R_CHIP-0603(1608-METRIC)
- R7: value 24.3K -> 143K; device Resistor:R_CHIP-0402(1005-METRIC) -> Resistor:R_CHIP-0603(1608-METRIC)
- R8: value 76.8K -> 4.7K
- R9: value 27.4K -> 3.65k; device Resistor:R_CHIP-0402(1005-METRIC) -> Resistor:R_CHIP-0603(1608-METRIC)
- U1: value MP2639AGR-Z -> AC103E2FAC_USS; device MP2639AGR-Z:MP2639AGR-Z -> 103AT‐2:AC103E2FAC_USS
- U2: value ATMEGA328P -> W25QXX128MBIT; device microbuilder:ATMEGA328P -> SparkFun-IC-Memory:W25QXX128MBIT-6X5-SKINNY_CENTER
- U4: value XC6209F332MR-GSOT-25_TOR -> TLV76633; device XC6209F332MR:XC6209F332MR-GSOT-25_TOR -> TLV76633:TLV76650QWDRBRQ1VSON_DRBRQ1_TEX
Connections:
- removed net ACOK: R6.2, U1.!ACLK, U2.(INT1)PD3
- removed net AD0: U2.(ADC0)PC0
- removed net AD1: U2.(ADC1)PC1
- removed net AD2: U2.(ADC2)PC2
- removed net AD3: U2.(ADC3)PC3
- removed net ILIM: R5.2
- removed net IO9: U2.(OC1)PB1
- removed net LED1: R16.1, U1.LED1
- removed net LED2: R17.1, U1.LED2
- removed net LED3: R18.1, U1.LED3
- removed net LED4: R19.1, U1.LED4
- removed net MODE: U1.MODE
- removed net PB: U1.!PB
- removed net VCC: C9.1, LED1.A, LED2.A, LED3.A, LED4.A, U1.VCC
- removed net VH: BT1.1, BT1.2, BT1.3, BT3.1, BT3.2, BT3.3, C14.1, C15.1, C17.1, J7.1, J7.2, J7.3, J7.4, U1.VH, U4.CE, U4.VIN
- new net 1.2V: IC1.DVDD, IC1.VREG_VOUT
- new net A2: IC1.GPIO28/AD2
- new net A3: IC1.GPIO29/AD3
- new net AVL: C9.1, R26.1, U7.AVL
- new net BAT+: BT1.1, BT1.2, BT1.3, BT11.1, BT11.2, BT12.1, BT12.2, BT3.1, BT3.2, BT3.3, C14.1, C15.1, U10.S, U10.S_2, U10.S_3
- new net BATSN: C11.2, U7.BATSN, U7.DISQBAT, U7.OTGEN
- new net BOOT: R30.2, RESET1.S, RESET1.S1
- new net CSINN: C3.2, C7.1, R5.1, U7.CSINN
- new net CSINP: C3.1, C8.1, R4.1, U7.CSINP
- new net DSG: Q1.D, R13.2, R18.1, U11.G
- new net EN_5V: IC1.GPIO25, U15.EN, U17.PC2(ADC2)
- new net EN_HAP: IC1.GPIO7, U13.EN, U17.PC0(ADC0)
- new net EN_LED: IC1.GPIO24, U17.PC1(ADC1), U8.SDB
- new net GAUGE: BT2.4, BT2.5, BT2.6, BT4.4, BT4.5, BT4.6, BT5.1, BT5.2, BT6.1, BT6.2, C28.1, C35.1, R15.2, R17.1, U12.2, U9.PWPD, U9.VSS
- new net INOKB: R6.1, TP13.1, U7.INOKB
- new net INTB: IC1.GPIO9, R8.1, TP14.1, TP3.1, U17.PD3(INT1), U7.INTB
- new net LX1: C22.1, U14.1, U7.LX1, U7.LX1_2, U7.LX1_3, U7.LX1_4
- new net LX2: C20.2, U14.2, U7.LX2, U7.LX2_2, U7.LX2_3
- new net MID: BT1.4, BT1.5, BT1.6, BT10.1, BT10.2, BT2.1, BT2.2, BT2.3, BT3.4, BT3.5, BT3.6, BT4.1, BT4.2, BT4.3, BT7.1, BT7.2, BT8.1, BT8.2, BT9.1, BT9.2, R25.1
- new net N$27: U10.D, U10.D_2, U10.D_3, U10.D_4, U11.D, U11.D_2, U11.D_3, U11.D_4
- new net N$28: C33.2, R19.2, R24.2
- new net N$29: CN1.1, U13.OUT+
- new net N$30: CN1.2, U13.OUT-
- new net N$31: C37.1, U13.REG
- new net N$32: C44.1, R9.2
- new net N$33: C45.1, R9.1, U15.COMP
- new net N$34: TP12.1, U4.SNS
- new net N$35: R28.2, R29.1, U15.VSENSE
- new net N$39: IC1.TESTEN
- new net NEOPIX: IC1.GPIO16
- new net NEO_PWR: IC1.GPIO17
- new net PACK+: C11.1, C29.2, C32.1, D4.A, Q1.S, R18.2, U11.S, U11.S_2, U11.S_3, U7.BATSP, U7.BATT, U7.BATT_2, U7.BATT_3, U9.PACK
- new net PH: C46.2, L1.2, U15.PH
- new net PVL: C10.1, R26.2, U7.INLIM, U7.ISET, U7.ITO, U7.PVL, U7.VSET
- new net QSPI_CS: IC1.!QSPI_CS, R30.1, R32.2, U2.!CS!
- new net QSPI_DATA[0]: IC1.QSPI_SD0, U2.D0/DI
- new net QSPI_DATA[1]: IC1.QSPI_SD1, U2.D1/DO
- new net QSPI_DATA[2]: IC1.QSPI_SD2, U2.D2/!WP!
- new net QSPI_DATA[3]: IC1.QSPI_SD3, U2.D3/!HOLD!
- new net QSPI_SCK: IC1.QSPI_SCLK, U2.CLK
- new net SRN: C31.1, R16.2, U9.SRN
- new net SRP: C31.2, R17.2, U9.SRP
- new net SWCLK: IC1.SWCLK, JP1.1
- new net SWDIO: IC1.SWDIO, JP1.2
- new net VC1: C34.1, C35.2, R25.2, U9.VC1
- new net VC2: C34.2, R24.1, U9.VC2
- new net VSYS: C12.1, C13.1, C16.1, C17.1, C38.1, C39.1, C40.1, C41.1, C42.1, C47.1, D4.C, J8.1, J8.2, J8.3, J8.4, U15.VIN, U4.EN, U4.IN, U7.SYS, U7.SYSA, U7.SYS_2, U7.SYS_3, U7.SYS_4, U7.SYS_5
- net +3.3V: now also C21.1, C27.2, C36.1, C48.2, C49.1, IC1.ADC_IOVDD, IC1.IOVDD, IC1.USB_IOVDD, IC1.VREG_IOVDD, R32.1, R6.2, R8.2, TP7.1, U13.VDD, U17.AVCC, U17.VCC@4, U17.VCC@6, U2.VDD, U4.NC_2, U4.OUT, U8.VCC; no longer TPR54.4, U2.AVCC, U2.VCC
- net +5V: now also C43.1, L1.1, R28.1; no longer C11.1, C2.1, C3.1, C4.1, C52.1, Q2.S_1, Q2.S_2, Q2.S_3, R8.2, R9.2, U1.VL
- net AREF: now also U17.AREF; no longer U2.AREF
- net CHG: now also R12.2, R19.1, U10.G; no longer U1.!CHG
- net D+: now also IC1.USB_D+, J1G$2.D+_B
- net D-: now also IC1.USB_D-, J1G$2.D-_B
- net DTR: now also TP11.1
- net EN/DVDD: now also IC1.GPIO27/AD1, U17.PB1(OC1A)
- net GND: now also C10.2, C12.2, C13.2, C16.2, C27.1, C30.1, C36.2, C37.2, C38.2, C39.2, C40.2, C41.2, C42.2, C43.2, C44.2, C45.2, C47.2, C48.1, C49.2, C8.2, IC1.GND, J7.1, J7.2, J7.3, J7.4, R11.1, R14.1, R15.1, R16.1, R29.2, RESET1.P, RESET1.P1, TP8.1, U1.2, U13.GND, U15.EPAD, U15.GND, U15.GND_2, U15.GND_3, U17.AGND, U17.GND@3, U17.GND@5, U4.GND, U4.GND_2, U4.THERMAL, U7.GND_2, U7.GND_3, U7.GND_4, U7.PGND, U7.PGND_2, U7.PGND_3, U7.PGND_4, U7.STBY, U8.EPAD, U8.GND; no longer C12.1, C3.2, C52.2, CIB.1, CTMR.1, D4.2, J8.1, J8.2, J8.3, J8.4, Q1.S, R4.1, RIB.2, RILIM.2, RISET.2, RNTC2.2, ROLIM.2, TPR54.3, U1.AGND, U1.PGND, U2.AGND, U4.VSS
- net IO2: now also IC1.GPIO8, TP5.1, U17.PD2(INT0); no longer TPR54.6, U2.(INT0)PD2
- net IO4: now also IC1.GPIO10, TP10.1, U17.PD4(XCK/T0); no longer TPR54.1, U2.(TO)PD4
- net IO5: now also IC1.GPIO11, TP9.1, U17.PD5(T1); no longer TPR54.2, U2.(T1)PD5
- net IO6: now also IC1.GPIO12, TP6.1, U17.PD6(AIN0); no longer TPR54.5, U2.(AIN0)PD6
- net IO7: now also IC1.GPIO13, TP4.1, U17.PD7(AIN1); no longer TPR54.7, U2.(AIN1)PD7
- net MISO: now also IC1.GPIO20, U17.PB4(MISO); no longer U2.(MISO)PB4
- net MOSI: now also IC1.GPIO19, U17.PB3(MOSI/OC2); no longer U2.(MOSI)PB3
- net N$1: now also C1.1, C2.1, R3.2, R5.2, U7.CHGIN, U7.CHGIN_2, U7.CHGIN_3, U7.CHGIN_4; no longer Q2.G, R6.1
- net N$10: now also U1.1, U7.THM; no longer CTMR.2, U1.TMR
- net N$11: now also D5.C, U8.OUT1; no longer C11.2, R7.2, R8.1, U1.FB
- net N$12: now also D6.C, U8.OUT2; no longer R10.2, R9.1, U1.VLIM
- net N$13: now also D7.C, U8.OUT3; no longer RNTC1.2, RNTC2.1, U1.NTC
- net N$14: now also D8.C, U8.!OUT4; no longer C12.2, RNTC1.1, U1.VNTC
- net N$15: now also D5.A, D6.A, D7.A, D8.A, U8.VOUT; no longer RILIM.1, U1.ILIM
- net N$16: now also R11.2, U8.AD; no longer RISET.1, U1.ISET
- net N$17: now also C25.1, U8.C1P; no longer ROLIM.1, U1.OLIM
- net N$18: now also C25.2, U8.C1N; no longer CIB.2, R11.2
- net N$19: now also R12.1, U9.CHG; no longer R11.1, RIB.1, U1.IB
- net N$2: now also C28.2, U9.PBI; no longer BT1.4, BT1.5, BT1.6, BT2.1, BT2.2, BT2.3
- net N$20: now also R13.1, U9.DSG; no longer LED3.C, R18.2
- net N$21: now also C29.1, C30.2; no longer LED4.C, R19.2
- net N$23: now also Q1.G, R14.2; no longer BT2.4, BT2.5, BT2.6, BT4.4, BT4.5, BT4.6
- net N$24: now also TP2.1, U13.IN_TRIG; no longer C21.1, U4.VOUT
- net N$25: now also C26.2, U8.C2P; no longer C1.1, J1G$2.D+_B, R3.2
- net N$26: now also C32.2, C33.1; no longer J1G$2.D-_B, Q1.G, R4.2
- net N$3: now also R7.2, U15.RT; no longer Q1.D, R5.1
- net N$4: now also U12.1, U9.T81; no longer BT3.4, BT3.5, BT3.6, BT4.1, BT4.2, BT4.3
- net N$5: now also C26.1, U8.C2N; no longer LED2.C, R17.2
- net N$6: now also R10.2, U8.ISET; no longer LED1.C, R16.2
- net N$7: now also C46.1, U15.BOOT; no longer C8.1, L1.1, U1.SW
- net N$8: now also C20.1, U7.BST2; no longer D4.1, L1.2, U1.LX
- net N$9: now also C22.2, U7.BST1; no longer C8.2, U1.BST
- net PDN: now also IC1.GPIO26/AD0, U17.PC3(ADC3)
- net RESET: now also IC1./RUN, U17.PC6(/RESET); no longer U2.RESET
- net RXD: now also IC1.GPIO1, U17.PD0(RXD); no longer U2.(RXD)PD0
- net SCK: now also IC1.GPIO18, U17.PB5(SCK); no longer U2.(SCK)PB5
- net SCL: now also IC1.GPIO3, U13.SCL, U17.PC5(ADC5/SCL), U7.SCL, U8.SCL, U9.SCL; no longer U2.(ADC5)PC5
- net SDA: now also IC1.GPIO2, U13.SDA, U17.PC4(ADC4/SDA), U7.SDA, U8.SDA, U9.SDA; no longer U2.(ADC4)PC4
- net SS: now also U17.PB2(SS/OC1B); no longer U2.(SS)PB2
- net TXD: now also IC1.GPIO0, U17.PD1(TXD); no longer U2.(TXD)PD1
- net VIN: now also C4.1, R4.2; no longer C7.1, Q2.D_1, Q2.D_2, Q2.D_3, Q2.D_4
- net VREG_IN: now also IC1.GPIO14, U17.PB0(ICP); no longer U2.(ICP)PB0
- net XTAL1: now also IC1.XOUT, R31.1, R31.2, U17.PB7(XTAL2/TOSC2); no longer U2.XTAL1
- net XTAL2: now also IC1.XIN, U17.PB6(XTAL1/TOSC1); no longer U2.XTAL2
Other:
- note added: "16MB Flash"
- note added: "2S2P / 10000mA / 18650"
- note added: "Alternative"
- note added: "BQ28Z610 - 2S Battery fuel gauge"
- note added: "CSTNE12M0G550000R0"
- note added: "DRV2605 - Haptic Controller"
- note added: "Disable flash boot (forces USB boot)"
- note added: "EN-DRV2605"
- note added: "EN-TPS54335"
- note added: "EN/DVDD"
- note added: "INTB"
- note added: "IS31FL3195 - LED DRIVER"
- note added: "MAX77962 - 2S CHARGER"
- note added: "PDN"
- note added: "ROB-08449"
- note added: "RP2040"
- note added: "SBD-LED Driver"
- note added: "TPR54 - Capacitive Sensor"
- note added: "TPS54335 - 5V Step-Down"
- note added: "TPS62056"
- note added: "TPS62111"
- note added: "TPS62162"
- note added: "TPS62172"
- note added: "TPS627431"
- note added: "TPS7A2633"
- note added: "XC6209F332"
- note added: "https://datasheets.maximintegrated.com/en/ds/MAX77962EVKIT-06-MAX77962EVKIT-12.pdf"
- note added: "https://www.ti.com/product/BQ28Z610#reference-designs"
- note added: "‎RLP4-200-500‎"
- note removed: "2.2uH"
- note removed: "2S1P / 5000mA / 18650, J2&J3 USED TO EXTEND THE BAT TO 10000mA"
- note removed: "4.5V/50mA"
- note removed: "ACOK"
- note removed: "BAT LED"
- note removed: "IRF7416PbF"
- note removed: "MP2639C"
- note removed: "RRH140P03TB1"
- note removed: "TPR54"
- note removed: "VCC can supply 50mA, *calculate LED resistor depending on Vf of LED"
- note removed: "https://www.azoteq.com/images/stories/pdf/proxsense_gpio_trackpad_datasheet.pdf"
- note removed: "https://www.monolithicpower.com/en/ev2639c-r-00a.html"
